File: HW/CAD/Eagle/DCF77_RX_1V0.sch (EAGLE design)
At the start: 39 parts, among them J131 2SK3557, J221 2SK3557, Q211 QT26V-77.000k, U271 LMH6645MF, X101 PHOENIX_1990067_1X8X2MM50_PTS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, X391 PHOENIX_1990067_1X8X2MM50_PTS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

Commit message: HW - Eagle - DCF77_RX_1V0 - value tweaks done
Parts:
- C111: value 10pF -> N/A
- C212: value 1.5pF -> 12pF
- C213: value EW_SGC3S100 -> SGC3S030NM
Other:
- note added: "1.8..4.5pF"
- note removed: "3.0..10pF"
Changed lines of the file:
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@@
 <part name="GND121" library="df4iah_supply" deviceset="GND" device=""/>
 <part name="X101" library="df4iah_connector" deviceset="PHOENIX_1990067_1X8X2MM50_PTSA-0-5" device=""/>
-<part name="C111" library="df4iah_rcl" deviceset="C-EU" device="C0402" value="10pF"/>
+<part name="C111" library="df4iah_rcl" deviceset="C-EU" device="C0402" value="N/A"/>
 <part name="C112" library="df4iah_c-trimm" deviceset="C-TRIMM__EW_SGC3S" device="" value="EW_SGC3S300"/>
 <part name="C122" library="df4iah_rcl" deviceset="C-EU" device="C0805" value="10nF"/>
@@
 <part name="GND201" library="df4iah_supply" deviceset="GND" device=""/>
 <part name="U271" library="df4iah_opamp" deviceset="LMH6645MF" device=""/>
-<part name="C213" library="df4iah_c-trimm" deviceset="C-TRIMM__EW_SGC3S" device="" value="EW_SGC3S100"/>
-<part name="C212" library="df4iah_rcl" deviceset="C-EU" device="C0402" value="1.5pF"/>
+<part name="C213" library="df4iah_c-trimm" deviceset="C-TRIMM__EW_SGC3S" device="" value="SGC3S030NM"/>
+<part name="C212" library="df4iah_rcl" deviceset="C-EU" device="C0402" value="12pF"/>
 <part name="GND251" library="df4iah_supply" deviceset="GND" device=""/>
 <part name="R251" library="df4iah_rcl" deviceset="R-EU_" device="R0805" value="1kR"/>
@@
 <text x="165.1" y="12.7" size="2.54" layer="97" ratio="15">Crystal, Driver &amp;
 Decider</text>
-<text x="71.12" y="93.98" size="1.778" layer="97">3.0..10pF</text>
+<text x="71.12" y="93.98" size="1.778" layer="97">1.8..4.5pF</text>
 <text x="22.86" y="162.56" size="2.54" layer="97" ratio="15">Crystal, Driver &amp; Decider</text>
 <text x="187.96" y="76.2" size="1.778" layer="94">A = 0 .. 40 dB</text>
